File: hardware/PCB Production/KICAD Files/Blue Line/Blue Line.kicad_pcb (KiCad board)
At the start: 2 copper layers, 203.2 x 254 mm, 25 parts, among them J1 Conn_01x03

Commit message: updating station_led_maps and blue line production files
Turns out ground planes are important ;) I definitely didn't forget to add one in the blue line PCB
Routing:
- added copper zone on B.Cu, net GND
